File: TKLC_v1/tklc_v1/tklc_v1.kicad_pcb (KiCad board)
At the start: 2 copper layers, 291 parts, among them J1 UART breakout for extension b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, J2 RGB Strip breakout, J3 Encoder breakout, SW1 CherryMX_LED, SW10 CherryMX_LED, SW11 CherryMX_LED, SW12 CherryMX_LED, SW13 CherryMX_LED, SW14 CherryMX_LED, SW15 CherryMX_LED, SW16 CherryMX_LED, SW17 RotaryEncoder_Switch, SW18 CherryMX_LED, SW19 CherryMX_LED, SW2 CherryMX_LED, SW20 CherryMX_LED, SW21 CherryMX_LED, SW22 CherryMX_LED, SW23 CherryMX_LED, SW24 CherryMX_LED, SW25 CherryMX_LED, SW26 CherryMX_LED, SW27 CherryMX_LED, SW28 CherryMX_LED, SW29 CherryMX_LED, SW3 CherryMX_LED, SW30 CherryMX_LED, SW31 CherryMX_LED, SW32 CherryMX_LED, SW33 CherryMX_LED, SW34 CherryMX_LED, SW35 CherryMX_LED, SW36 CherryMX_LED, SW37 CherryMX_LED, SW38 CherryMX_LED, SW39 CherryMX_LED, SW4 CherryMX_LED, SW40 CherryMX_LED, SW41 CherryMX_LED, SW42 CherryMX_LED, SW43 CherryMX_LED, SW44 CherryMX_LED, SW45 CherryMX_LED, SW46 CherryMX_LED, SW47 CherryMX_LED, SW48 CherryMX_LED, SW49 CherryMX_LED, SW5 CherryMX_LED, SW50 CherryMX_LED, SW51 CherryMX_LED, SW52 CherryMX_LED, SW53 CherryMX_LED, SW54 CherryMX_LED, SW55 CherryMX_LED, SW56 CherryMX_LED, SW57 CherryMX_LED, SW58 CherryMX_LED, SW59 CherryMX_LED, SW6 CherryMX_LED, SW60 CherryMX_LED, SW61 CherryMX_LED, SW62 CherryMX_LED, SW63 CherryMX_LED, SW64 CherryMX_LED, SW65 CherryMX_LED, SW66 CherryMX_LED, SW67 CherryMX_LED, SW68 CherryMX_LED, SW69 CherryMX_LED, SW7 CherryMX_LED, SW70 CherryMX_LED, SW71 CherryMX_LED, SW72 CherryMX_LED, SW73 CherryMX_LED, SW74 CherryMX_LED, SW75 CherryMX_LED, SW76 CherryMX_LED, SW77 CherryMX_LED, SW78 CherryMX_LED, SW79 CherryMX_LED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

Commit message: Finished laying out PCB
Parts:
- R1, R10, R11, R12, R13, R14, R15, R16, R18, R19, R2, R20, R21, R22, R23, R24, R25, R26, R27, R28, R29, R3, R30, R31, R32, R33, R34, R35, R36, R37, R38, R39, R4, R40, R41, R42, R43, R44, R45, R46, R47, R48, R49, R5, R50, R51, R52, R53, R54, R55, R56, R57, R58, R59, R6, R60, R61, R62, R63, R64, R65, R66, R67, R68, R69, R7, R70, R71, R72, R73, R74, R75, R76, R77, R78, R79, R8, R80, R81, R82, R83, R84, R85, R86, R87, R88, R89, R9, R90, R91, R92: footprint Resistor_THT:R_Axial_DIN0207_L6.3mm_D2.5mm_P7.62mm_Horizontal -> edited_footprints:R_Axial_DIN0207_L6.3mEDIT_m_D2.5mm_P7.62mm_Horizontal
- SW17: footprint Rotary_Encoder:RotaryEncoder_Alps_EC11E-Switch_Vertical_H20mm -> edited_footprints:EDIT_RotaryEncoder_Alps_EC11E-Switch_Vertical_H20mm
- moved R1 444.5 mm to (59.5, 121.4), turned to 180 degrees
- moved R35 420.9 mm to (78.6, 145.3), turned to 180 degrees
- moved R20 403.6 mm to (97.6, 126.2), turned to 180 degrees
- moved D2 401.3 mm to (88.1, 121.4), turned to 90 degrees
- moved R2 394.1 mm to (78.6, 121.4), turned to 180 degrees
- moved D51 384.6 mm to (102.4, 183.4), turned to 90 degrees
- moved R67 381.8 mm to (111.9, 183.4), turned to 180 degrees
- moved D20 381.7 mm to (107.2, 145.3), turned to 90 degrees
- moved D35 376.8 mm to (97.6, 164.3), turned to 90 degrees
- moved R50 375.6 mm to (64.3, 164.3), turned to 180 degrees
- moved R34 371.7 mm to (59.5, 145.3), turned to 180 degrees
- moved R65 371.3 mm to (71.4, 183.4), turned to 180 degrees
- moved D5 370.4 mm to (145.3, 121.4), turned to 90 degrees
- moved R18 364.1 mm to (59.5, 126.2), turned to 180 degrees
- moved D37 361.0 mm to (135.7, 164.3), turned to 90 degrees
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Routing:
- added copper zone on F.Cu, net GND
Other:
- board outline added: 332.6 x 146.9 mm
