File: TKLC_v1/tklc_v1/tklc_v1.kicad_sch (KiCad schematic)
At the start: 93 parts, among them U1 WeAct-RP2040-Pico

Commit message: Add files via upload
Parts:
- removed SW? (x91): CherryMX_LED, symbol Cherry MX:CherryMX_LED
- added D? (x92): 1N4148, Diode_THT:D_DO-35_SOD27_P7.62mm_Horizontal, symbol Diode:1N4148
- added SW? (x91): CherryMX_LED, symbol Cherry MX:CherryMX_LED
Connections:
- net at SW?.3 (K): now also D?.2 (A)
- new net: D?.2 (A), SW?.3 (K) (x91)
Other:
- moved on the sheet: SW?, U1

Commit message: Add files via upload
Parts:
- removed D? (x91): 1N4148, Diode_THT:D_DO-35_SOD27_P7.62mm_Horizontal, symbol Diode:1N4148
- removed SW? (x91): CherryMX_LED, symbol Cherry MX:CherryMX_LED
- added D10, D11, D12, D13, D14, D15, D16, D17, D18, D19, D2, D20, D21, D22, D23, D24, D25, D26, D27, D28, D29, D3, D30, D31, D32, D33, D34, D35, D36, D37, D38, D39, D4, D40, D41, D42, D43, D44, D45, D46, D47, D48, D49, D5, D50, D51, D52, D53, D54, D55, D56, D57, D58, D59, D6, D60, D61, D62, D63, D64, D65, D66, D67, D68, D69, D7, D70, D71, D72, D73, D74, D75, D76, D77, D78, D79, D8, D80, D81, D82, D83, D84, D85, D86, D87, D88, D89, D9, D90, D91, D92: 1N4148, Diode_THT:D_DO-35_SOD27_P7.62mm_Horizontal, symbol Diode:1N4148
- added SW10, SW11, SW12, SW13, SW14, SW15, SW16, SW17, SW18, SW19, SW2, SW20, SW21, SW22, SW23, SW24, SW25, SW26, SW27, SW28, SW29, SW3, SW30, SW31, SW32, SW33, SW34, SW35, SW36, SW37, SW38, SW39, SW4, SW40, SW41, SW42, SW43, SW44, SW45, SW46, SW47, SW48, SW49, SW5, SW50, SW51, SW52, SW53, SW54, SW55, SW56, SW57, SW58, SW59, SW6, SW60, SW61, SW62, SW63, SW64, SW65, SW66, SW67, SW68, SW69, SW7, SW70, SW71, SW72, SW73, SW74, SW75, SW76, SW77, SW78, SW79, SW8, SW80, SW81, SW82, SW83, SW84, SW85, SW86, SW87, SW88, SW89, SW9, SW90, SW91, SW92: CherryMX_LED, symbol Cherry MX:CherryMX_LED
- gave numbers to parts that had none: 2
Connections:
- net row0: now reaches D1.1 (K)
- net row0: now also U1.20 (GP15), D10.1 (K), D11.1 (K), D12.1 (K), D13.1 (K), D14.1 (K), D15.1 (K), D16.1 (K), D17.1 (K), D2.1 (K), D3.1 (K), D4.1 (K), D5.1 (K), D6.1 (K), D7.1 (K), D8.1 (K), D9.1 (K)
- net at D1.2 (A): now also SW1.1; no longer SW1.3 (K)
- net col16: now reaches U1.1 (GP0)
- net col16: now also SW17.2, SW33.2, SW49.2, SW64.2, SW78.2, SW92.2
- net row5: now reaches U1.14 (GP10)
- net row5: now also D79.1 (K), D80.1 (K), D81.1 (K), D82.1 (K), D83.1 (K), D84.1 (K), D85.1 (K), D86.1 (K), D87.1 (K), D88.1 (K), D89.1 (K), D90.1 (K), D91.1 (K), D92.1 (K)
- net row4: now reaches U1.15 (GP11)
- net row4: now also D65.1 (K), D66.1 (K), D67.1 (K), D68.1 (K), D69.1 (K), D70.1 (K), D71.1 (K), D72.1 (K), D73.1 (K), D74.1 (K), D75.1 (K), D76.1 (K), D77.1 (K), D78.1 (K)
- net row3: now reaches U1.16 (GP12)
- net row3: now also D50.1 (K), D51.1 (K), D52.1 (K), D53.1 (K), D54.1 (K), D55.1 (K), D56.1 (K), D57.1 (K), D58.1 (K), D59.1 (K), D60.1 (K), D61.1 (K), D62.1 (K), D63.1 (K), D64.1 (K)
- net row2: now reaches U1.17 (GP13)
- net row2: now also D34.1 (K), D35.1 (K), D36.1 (K), D37.1 (K), D38.1 (K), D39.1 (K), D40.1 (K), D41.1 (K), D42.1 (K), D43.1 (K), D44.1 (K), D45.1 (K), D46.1 (K), D47.1 (K), D48.1 (K), D49.1 (K)
- net row1: now reaches U1.19 (GP14)
- net row1: now also D18.1 (K), D19.1 (K), D20.1 (K), D21.1 (K), D22.1 (K), D23.1 (K), D24.1 (K), D25.1 (K), D26.1 (K), D27.1 (K), D28.1 (K), D29.1 (K), D30.1 (K), D31.1 (K), D32.1 (K), D33.1 (K)
- net col0: now reaches U1.21 (GP16)
- net col0: now also SW1.2, SW18.2, SW34.2, SW50.2, SW65.2, SW79.2
- net col1: now reaches U1.22 (GP17)
- net col1: now also SW19.2, SW2.2, SW35.2, SW51.2, SW80.2
- net col2: now reaches U1.24 (GP18)
- net col2: now also SW20.2, SW3.2, SW36.2, SW52.2, SW66.2, SW81.2
- net col3: now reaches U1.25 (GP19)
- net col3: now also SW21.2, SW37.2, SW4.2, SW53.2, SW67.2, SW82.2
- net col4: now reaches U1.26 (GP20)
- net col4: now also SW22.2, SW38.2, SW5.2, SW54.2, SW68.2
- net col5: now reaches U1.27 (GP21)
- net col5: now also SW23.2, SW39.2, SW55.2, SW6.2, SW69.2, SW83.2
- net col6: now reaches U1.29 (GP22)
- net col6: now also SW24.2, SW40.2, SW56.2, SW7.2, SW70.2, SW84.2
- net col7: now reaches U1.30 (GP26)
- net col7: now also SW25.2, SW41.2, SW57.2, SW71.2, SW8.2, SW85.2
- net col8: now reaches U1.31 (GP27)
- net col8: now also SW26.2, SW42.2, SW58.2, SW72.2, SW9.2
- net col9: now reaches U1.32 (GP28)
- net col9: now also SW10.2, SW27.2, SW43.2, SW59.2, SW73.2, SW86.2
- net col10: now reaches U1.34 (GP29)
- net col10: now also SW11.2, SW28.2, SW44.2, SW60.2, SW74.2, SW87.2
- net col11: now reaches U1.35 (ADC_VREF)
- net col11: now also SW12.2, SW29.2, SW45.2, SW61.2, SW75.2
- net col12: now reaches U1.36 (GP24)
- net col13: now reaches U1.37 (3V3)
- net col13: now also SW14.2, SW62.2, SW76.2, SW89.2
- net col14: now reaches U1.39 (VSYS)
- net col14: now also SW15.2, SW31.2, SW47.2, SW90.2
- net col15: now reaches U1.40 (VBUS)
- net col15: now also SW16.2, SW32.2, SW48.2, SW63.2, SW77.2, SW91.2
- new net: D8.2 (A), SW8.1
- new net: D11.2 (A), SW11.1
- new net: D66.2 (A), SW66.1
- new net: D61.2 (A), SW61.1
- new net: D50.2 (A), SW50.1
- new net: D19.2 (A), SW19.1
- new net: D43.2 (A), SW43.1
- new net: D24.2 (A), SW24.1
- new net: D62.2 (A), SW62.1
- new net: D40.2 (A), SW40.1
- new net: D14.2 (A), SW14.1
- new net: D49.2 (A), SW49.1
- new net: D15.2 (A), SW15.1
- new net: D79.2 (A), SW79.1
- new net: D27.2 (A), SW27.1
- new net: D44.2 (A), SW44.1
- new net: D42.2 (A), SW42.1
- new net: D85.2 (A), SW85.1
- new net: D60.2 (A), SW60.1
- new net: D92.2 (A), SW92.1
- new net: D51.2 (A), SW51.1
- new net: D5.2 (A), SW5.1
- new net: D76.2 (A), SW76.1
- new net: D64.2 (A), SW64.1
- new net: D82.2 (A), SW82.1
- new net: D3.2 (A), SW3.1
- new net: D25.2 (A), SW25.1
- new net: D78.2 (A), SW78.1
- new net: D80.2 (A), SW80.1
- new net: D88.2 (A), SW88.1
- new net: D33.2 (A), SW33.1
- new net: D67.2 (A), SW67.1
- new net: D39.2 (A), SW39.1
- new net: D10.2 (A), SW10.1
- new net: D59.2 (A), SW59.1
- new net: D38.2 (A), SW38.1
- new net: D34.2 (A), SW34.1
- new net: D77.2 (A), SW77.1
- new net: D69.2 (A), SW69.1
- new net: D28.2 (A), SW28.1
- new net: D7.2 (A), SW7.1
- new net: D6.2 (A), SW6.1
- new net: SW13.2, SW30.2, SW46.2, SW88.2
- new net: D58.2 (A), SW58.1
- new net: D41.2 (A), SW41.1
- new net: D72.2 (A), SW72.1
- new net: D90.2 (A), SW90.1
- new net: D83.2 (A), SW83.1
- new net: D84.2 (A), SW84.1
- new net: D26.2 (A), SW26.1
- new net: D18.2 (A), SW18.1
- new net: D74.2 (A), SW74.1
- new net: D56.2 (A), SW56.1
- new net: D32.2 (A), SW32.1
- new net: D45.2 (A), SW45.1
- new net: D55.2 (A), SW55.1
- new net: D73.2 (A), SW73.1
- new net: D35.2 (A), SW35.1
- new net: D37.2 (A), SW37.1
- new net: D46.2 (A), SW46.1
- new net: D86.2 (A), SW86.1
- new net: D70.2 (A), SW70.1
- new net: D2.2 (A), SW2.1
- new net: D63.2 (A), SW63.1
- new net: D20.2 (A), SW20.1
- new net: D22.2 (A), SW22.1
- new net: D31.2 (A), SW31.1
- new net: D30.2 (A), SW30.1
- new net: D81.2 (A), SW81.1
- new net: D65.2 (A), SW65.1
- new net: D89.2 (A), SW89.1
- new net: D48.2 (A), SW48.1
- new net: D91.2 (A), SW91.1
- new net: D87.2 (A), SW87.1
- new net: D17.2 (A), SW17.1
- new net: D23.2 (A), SW23.1
- new net: D9.2 (A), SW9.1
- new net: D54.2 (A), SW54.1
- new net: D13.2 (A), SW13.1
- new net: D71.2 (A), SW71.1
- new net: D53.2 (A), SW53.1
- new net: D21.2 (A), SW21.1
- new net: D57.2 (A), SW57.1
- new net: D29.2 (A), SW29.1
- new net: D68.2 (A), SW68.1
- new net: D36.2 (A), SW36.1
- new net: D12.2 (A), SW12.1
- new net: D4.2 (A), SW4.1
- new net: D47.2 (A), SW47.1
- new net: D52.2 (A), SW52.1
- new net: D16.2 (A), SW16.1
- new net: D75.2 (A), SW75.1
- no-connect marks 0 -> 9
Other:
- moved on the sheet: D1, SW1, U1

Commit message: Add files via upload
Parts:
- removed SW17: CherryMX_LED, symbol Cherry MX:CherryMX_LED
- added D77: 1N4148, Diode_THT:D_DO-35_SOD27_P7.62mm_Horizontal, symbol Diode:1N4148
- added SW17: RotaryEncoder_Switch, symbol Device:RotaryEncoder_Switch
- added SW77: CherryMX_LED, symbol Cherry MX:CherryMX_LED
- renumbered D77 to D78, D78 to D79, D79 to D80, D80 to D81, D81 to D82, D82 to D83, D83 to D84, D84 to D85, D85 to D86, D86 to D87, D87 to D88, D88 to D89, D89 to D90, D90 to D91, D91 to D92, D92 to D93, SW77 to SW78, SW78 to SW79, SW79 to SW80, SW80 to SW81, SW81 to SW82, SW82 to SW83, SW83 to SW84, SW84 to SW85, SW85 to SW86, SW86 to SW87, SW87 to SW88, SW88 to SW89, SW89 to SW90, SW90 to SW91, SW91 to SW92, SW92 to SW93
Connections:
- net GND: now also SW17.C
- net col0: now also U1.1 (GP0); no longer U1.21 (GP16)
- net col1: now also U1.2 (GP1); no longer U1.22 (GP17)
- net col10: now also U1.14 (GP10); no longer U1.34 (GP29)
- net col11: now also U1.15 (GP11); no longer U1.35 (ADC_VREF)
- net col12: now also U1.16 (GP12); no longer U1.36 (GP24)
- net col13: now also U1.17 (GP13); no longer U1.37 (3V3)
- net col14: now also U1.19 (GP14), SW77.2; no longer U1.39 (VSYS)
- net col15: now also U1.20 (GP15); no longer U1.40 (VBUS)
- net col16: now also U1.21 (GP16), SW17.S1; no longer U1.1 (GP0)
- net col2: now also U1.4 (GP2); no longer U1.24 (GP18)
- net col3: now also U1.5 (GP3); no longer U1.25 (GP19)
- net col4: now also U1.6 (GP4); no longer U1.26 (GP20)
- net col5: now also U1.7 (GP5); no longer U1.27 (GP21)
- net col6: now also U1.9 (GP6); no longer U1.29 (GP22)
- net col7: now also U1.10 (GP7); no longer U1.30 (GP26)
- net col8: now also U1.11 (GP8); no longer U1.31 (GP27)
- net col9: now also U1.12 (GP9); no longer U1.32 (GP28)
- net row0: now also U1.26 (GP20); no longer U1.20 (GP15)
- net row1: now also U1.27 (GP21); no longer U1.19 (GP14)
- net row2: now also U1.29 (GP22); no longer U1.17 (GP13)
- net row3: now also U1.30 (GP26); no longer U1.16 (GP12)
- net row4: now also U1.31 (GP27), D77.1 (K); no longer U1.15 (GP11)
- net row5: now also U1.32 (GP28); no longer U1.14 (GP10)
- net at D17.2 (A): now also SW17.S2
- new net: D77.2 (A), SW77.1
- new net EncoderA: SW17.A, U1.25 (GP19)
- new net EncoderB: SW17.B, U1.24 (GP18)
- new net LED_CONTROL: U1.34 (GP29)
- new net RGB_DATA: U1.22 (GP17)
- new net UART_CONNECT: U1.36 (GP24)
- no-connect marks 9 -> 0
Other:
- moved on the sheet: D1, D10, D11, D12, D13, D14, D15, D16, D17, D2, D3, D33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

Commit message: Add files via upload
Parts:
- removed D85: 1N4148, Diode_THT:D_DO-35_SOD27_P7.62mm_Horizontal, symbol Diode:1N4148
- removed SW85: CherryMX_LED, symbol Cherry MX:CherryMX_LED
- added R1, R10, R11, R12, R13, R14, R15, R16, R18, R19, R2, R20, R21, R22, R23, R24, R25, R26, R27, R28, R29, R3, R30, R31, R32, R33, R34, R35, R36, R37, R38, R39, R4, R40, R41, R42, R43, R44, R45, R46, R47, R48, R49, R5, R50, R51, R52, R53, R54, R55, R56, R57, R58, R59, R6, R60, R61, R62, R63, R64, R65, R66, R67, R68, R69, R7, R70, R71, R72, R73, R74, R75, R76, R77, R78, R79, R8, R80, R81, R82, R83, R84, R85, R86, R87, R88, R89, R9, R90, R91, R92: RLED, symbol Device:R
- added U10, U11, U12, U13, U2, U3, U4, U5, U6, U7, U8, U9: MC34064P, Package_TO_SOT_THT:TO-92L_Inline, symbol Power_Supervisor:MC34064P
- renumbered D86 to D85, D87 to D86, D88 to D87, D89 to D88, D90 to D89, D91 to D90, D92 to D91, D93 to D92, SW86 to SW85, SW87 to SW86, SW88 to SW87, SW89 to SW88, SW90 to SW89, SW91 to SW90, SW92 to SW91, SW93 to SW92
Connections:
- net EncoderA: now also U1.36 (GP24); no longer U1.25 (GP19)
- net EncoderB: now also U1.34 (GP29); no longer U1.24 (GP18)
- net GND: now also U11.3 (GND), U13.3 (GND), U3.3 (GND), U5.3 (GND), U7.3 (GND), U9.3 (GND); no longer U1.41 (GND)
- net LED_CONTROL: now also U1.24 (GP18), U11.2 (IN), U13.2 (IN), U3.2 (IN), U5.2 (IN), U7.2 (IN), U9.2 (IN); no longer U1.34 (GP29)
- net UART_CONNECT: now also U1.25 (GP19); no longer U1.36 (GP24)
- net row0: now also U2.2 (IN)
- net row1: now also U4.2 (IN)
- net row2: now also U6.2 (IN)
- net row3: now also U8.2 (IN)
- net row4: now also U10.2 (IN)
- net row5: now also U12.2 (IN)
- net at SW61.3 (K): now also R61.2
- net LED_3_IN: now reaches SW61.4 (A)
- net LED_3_IN: now also SW34.4 (A), SW35.4 (A), SW50.4 (A), SW51.4 (A), SW52.4 (A), SW53.4 (A), SW54.4 (A), SW55.4 (A), SW56.4 (A), SW57.4 (A), SW58.4 (A), SW59.4 (A), SW60.4 (A), SW62.4 (A), U8.3 (GND)
- net at SW50.3 (K): now also R50.2
- net at SW19.3 (K): now also R19.2
- net LED_1_IN: now reaches SW19.4 (A)
- net LED_1_IN: now also SW16.4 (A), SW18.4 (A), SW20.4 (A), SW21.4 (A), SW22.4 (A), SW23.4 (A), SW24.4 (A), SW25.4 (A), SW26.4 (A), SW27.4 (A), SW28.4 (A), SW29.4 (A), SW30.4 (A), SW31.4 (A), SW32.4 (A), U4.3 (GND)
- net at SW62.3 (K): now also R62.2
- net at SW40.3 (K): now also R40.2
- net LED_2_IN: now reaches SW40.4 (A)
- net LED_2_IN: now also SW33.4 (A), SW36.4 (A), SW37.4 (A), SW38.4 (A), SW39.4 (A), SW41.4 (A), SW42.4 (A), SW43.4 (A), SW44.4 (A), SW45.4 (A), SW46.4 (A), SW47.4 (A), SW48.4 (A), SW49.4 (A), U6.3 (GND)
- net at SW14.3 (K): now also R14.2
- net LED_0_IN: now reaches SW14.4 (A)
- net LED_0_IN: now also SW1.4 (A), SW10.4 (A), SW11.4 (A), SW12.4 (A), SW13.4 (A), SW15.4 (A), SW2.4 (A), SW3.4 (A), SW4.4 (A), SW5.4 (A), SW6.4 (A), SW7.4 (A), SW8.4 (A), SW9.4 (A), U2.3 (GND)
- net at SW80.3 (K): now also R80.2
- net LED_5_IN: now reaches SW80.4 (A)
- net LED_5_IN: now also SW65.4 (A), SW66.4 (A), SW81.4 (A), SW82.4 (A), SW83.4 (A), SW84.4 (A), SW85.4 (A), SW86.4 (A), SW87.4 (A), SW88.4 (A), SW89.4 (A), SW90.4 (A), SW91.4 (A), SW92.4 (A), U12.3 (GND)
- net at SW44.3 (K): now also R44.2
- net at SW42.3 (K): now also R42.2
- net at SW85.3 (K): now also R85.2
- net at SW51.3 (K): now also R51.2
- net at SW64.3 (K): now also R64.2
- net LED_4_IN: now reaches SW64.4 (A)
- net LED_4_IN: now also SW63.4 (A), SW67.4 (A), SW68.4 (A), SW69.4 (A), SW70.4 (A), SW71.4 (A), SW72.4 (A), SW73.4 (A), SW74.4 (A), SW75.4 (A), SW76.4 (A), SW77.4 (A), SW78.4 (A), SW79.4 (A), U10.3 (GND)
- net at SW3.3 (K): now also R3.2
- net at SW25.3 (K): now also R25.2
- net at SW79.3 (K): now also R79.2
- net at SW81.3 (K): now also R81.2
- net at SW43.3 (K): now also R43.2
- net at SW39.3 (K): now also R39.2
- net at SW11.3 (K): now also R11.2
- net at SW34.3 (K): now also R34.2
- net at SW15.3 (K): now also R15.2
- net at SW69.3 (K): now also R69.2
- net at SW28.3 (K): now also R28.2
- net at SW77.3 (K): now also R77.2
- net at SW88.3 (K): now also R88.2
- net at SW58.3 (K): now also R58.2
- net at SW38.3 (K): now also R38.2
- net at SW90.3 (K): now also R90.2
- net at SW84.3 (K): now also R84.2
- net at SW26.3 (K): now also R26.2
- net at SW74.3 (K): now also R74.2
- net at SW56.3 (K): now also R56.2
- net at SW76.3 (K): now also R76.2
- net at SW86.3 (K): now also R86.2
- net at SW59.3 (K): now also R59.2
- net at SW2.3 (K): now also R2.2
- net at SW63.3 (K): now also R63.2
- net at SW20.3 (K): now also R20.2
- net ADC_VREF: now reaches U1.35 (ADC_VREF)
- net 3V3: now reaches U1.37 (3V3)
- net VSYS: now reaches U1.39 (VSYS)
- net VSYS: now also U10.1 (~{RESET}), U12.1 (~{RESET}), U2.1 (~{RESET}), U4.1 (~{RESET}), U6.1 (~{RESET}), U8.1 (~{RESET})
- net VBUS: now reaches U1.40 (VBUS)
- net at SW31.3 (K): now also R31.2
- net at SW8.3 (K): now also R8.2
- net at SW65.3 (K): now also R65.2
- net at SW66.3 (K): now also R66.2
- net at SW24.3 (K): now also R24.2
- net at SW48.3 (K): now also R48.2
- net at SW87.3 (K): now also R87.2
- net at SW70.3 (K): now also R70.2
- net at SW67.3 (K): now also R67.2
- net at SW89.3 (K): now also R89.2
- net at SW73.3 (K): now also R73.2
- net at SW54.3 (K): now also R54.2
- net at SW30.3 (K): now also R30.2
- net at SW71.3 (K): now also R71.2
- net at SW10.3 (K): now also R10.2
- net at SW53.3 (K): now also R53.2
- net at SW83.3 (K): now also R83.2
- net at SW35.3 (K): now also R35.2
- net at SW21.3 (K): now also R21.2
- net at SW32.3 (K): now also R32.2
- net at SW72.3 (K): now also R72.2
- net at SW57.3 (K): now also R57.2
- net at SW91.3 (K): now also R91.2
- net at SW41.3 (K): now also R41.2
- net at SW29.3 (K): now also R29.2
- net at SW92.3 (K): now also R92.2
- net at SW68.3 (K): now also R68.2
- net at SW60.3 (K): now also R60.2
- net at SW78.3 (K): now also R78.2
- net at SW36.3 (K): now also R36.2
- net at SW45.3 (K): now also R45.2
- net at SW4.3 (K): now also R4.2
- net at SW13.3 (K): now also R13.2
- net at SW5.3 (K): now also R5.2
- net at SW12.3 (K): now also R12.2
- net at SW52.3 (K): now also R52.2
- net at SW23.3 (K): now also R23.2
- net at SW9.3 (K): now also R9.2
- net at SW82.3 (K): now also R82.2
- net at SW6.3 (K): now also R6.2
- net at SW16.3 (K): now also R16.2
- net at SW1.3 (K): now also R1.2
- net at SW49.3 (K): now also R49.2
- net at SW18.3 (K): now also R18.2
- net at SW7.3 (K): now also R7.2
- net at SW27.3 (K): now also R27.2
- net at SW37.3 (K): now also R37.2
- net at SW55.3 (K): now also R55.2
- net at SW33.3 (K): now also R33.2
- net at SW47.3 (K): now also R47.2
- net at SW75.3 (K): now also R75.2
- net at SW22.3 (K): now also R22.2
- net at SW46.3 (K): now also R46.2
- net col12 renamed LED_0_OUT
- net LED_0_OUT: now also R1.1, R10.1, R11.1, R12.1, R13.1, R14.1, R15.1, R2.1, R3.1, R4.1, R5.1, R6.1, R7.1, R8.1, R9.1, U3.1 (~{RESET})
- new net LED_1_OUT: R16.1, R18.1, R19.1, R20.1, R21.1, R22.1, R23.1, R24.1, R25.1, R26.1, R27.1, R28.1, R29.1, R30.1, R31.1, R32.1, U5.1 (~{RESET})
- new net LED_2_OUT: R33.1, R36.1, R37.1, R38.1, R39.1, R40.1, R41.1, R42.1, R43.1, R44.1, R45.1, R46.1, R47.1, R48.1, R49.1, U7.1 (~{RESET})
- new net LED_3_OUT: R34.1, R35.1, R50.1, R51.1, R52.1, R53.1, R54.1, R55.1, R56.1, R57.1, R58.1, R59.1, R60.1, R61.1, R62.1, U9.1 (~{RESET})
- new net LED_4_OUT: R63.1, R64.1, R67.1, R68.1, R69.1, R70.1, R71.1, R72.1, R73.1, R74.1, R75.1, R76.1, R77.1, R78.1, R79.1, U11.1 (~{RESET})
- new net LED_5_OUT: R65.1, R66.1, R80.1, R81.1, R82.1, R83.1, R84.1, R85.1, R86.1, R87.1, R88.1, R89.1, R90.1, R91.1, R92.1, U13.1 (~{RESET})
Other:
- moved on the sheet: U1

Commit message: Add files via upload
Parts:
- added J1: UART breakout for extension board, Connector:FanPinHeader_1x03_P2.54mm_Vertical, symbol Connector:Conn_01x03_Female
- added J2: RGB Strip breakout, Connector:FanPinHeader_1x03_P2.54mm_Vertical, symbol Connector:Conn_01x03_Female
- added J3: Encoder breakout, Connector:FanPinHeader_1x04_P2.54mm_Vertical, symbol Connector:Conn_01x04_Female
- R1, R10, R11, R12, R13, R14, R15, R16, R18, R19, R2, R20, R21, R22, R23, R24, R25, R26, R27, R28, R29, R3, R30, R31, R32, R33, R34, R35, R36, R37, R38, R39, R4, R40, R41, R42, R43, R44, R45, R46, R47, R48, R49, R5, R50, R51, R52, R53, R54, R55, R56, R57, R58, R59, R6, R60, R61, R62, R63, R64, R65, R66, R67, R68, R69, R7, R70, R71, R72, R73, R74, R75, R76, R77, R78, R79, R8, R80, R81, R82, R83, R84, R85, R86, R87, R88, R89, R9, R90, R91, R92: footprint (none) -> Resistor_THT:R_Axial_DIN0207_L6.3mm_D2.5mm_P7.62mm_Horizontal
- SW1, SW10, SW11, SW12, SW13, SW14, SW15, SW16, SW18, SW19, SW2, SW20, SW21, SW22, SW23, SW24, SW25, SW26, SW27, SW28, SW29, SW3, SW30, SW32, SW33, SW35, SW36, SW37, SW38, SW39, SW4, SW40, SW41, SW42, SW43, SW44, SW45, SW46, SW48, SW49, SW5, SW51, SW52, SW53, SW54, SW55, SW56, SW57, SW58, SW59, SW6, SW60, SW61, SW63, SW64, SW66, SW67, SW68, SW69, SW7, SW70, SW71, SW72, SW73, SW74, SW75, SW77, SW78, SW79, SW8, SW81, SW82, SW83, SW89, SW9, SW90, SW91, SW92: footprint (none) -> CherrryMX_PCB_Kailh_LED:CherryMX_1.00u_PCB_KailhSocket_LED
- SW17: footprint (none) -> Rotary_Encoder:RotaryEncoder_Alps_EC11E-Switch_Vertical_H20mm
- SW31: footprint (none) -> CherryMX_PCB_Kailh_StabTop_LED:CherryMX_2.00u_PCB_KailhSocket_StabWireTop_LED
- SW34, SW47: footprint (none) -> CherrryMX_PCB_Kailh_LED:CherryMX_1.50u_PCB_KailhSocket_LED
- SW50, SW76: footprint (none) -> CherrryMX_PCB_Kailh_LED:CherryMX_1.75u_PCB_KailhSocket_LED
- SW62, SW65, SW85: footprint (none) -> CherryMX_PCB_Kailh_StabTop_LED:CherryMX_2.25u_PCB_KailhSocket_StabWireTop_LED
- SW80, SW86, SW87, SW88: footprint (none) -> CherrryMX_PCB_Kailh_LED:CherryMX_1.25u_PCB_KailhSocket_LED
- SW84: footprint (none) -> CherryMX_PCB_Kailh_StabTop_LED:CherryMX_2.75u_PCB_KailhSocket_StabWireTop_LED
- U1: footprint (none) -> WeAct-RP2040-Pico:WeAct-RP2040-Pico
Connections:
- net 3V3: now also J1.3 (Pin_3)
- net EncoderA: now also J3.1 (Pin_1)
- net EncoderB: now also J3.2 (Pin_2)
- net GND: now also J1.1 (Pin_1), J2.1 (Pin_1)
- net RGB_DATA: now also J2.3 (Pin_3)
- net UART_CONNECT: now also J1.2 (Pin_2)
- net VBUS: now also J2.2 (Pin_2)
- net col16: now also J3.3 (Pin_3)
- net row0: now also J3.4 (Pin_4)
Other:
- title: (none) -> TKL Compact Mechanical Keyboard

Commit message: Finished laying out PCB
Parts:
- R1, R10, R11, R12, R13, R14, R15, R16, R18, R19, R2, R20, R21, R22, R23, R24, R25, R26, R27, R28, R29, R3, R30, R31, R32, R33, R34, R35, R36, R37, R38, R39, R4, R40, R41, R42, R43, R44, R45, R46, R47, R48, R49, R5, R50, R51, R52, R53, R54, R55, R56, R57, R58, R59, R6, R60, R61, R62, R63, R64, R65, R66, R67, R68, R69, R7, R70, R71, R72, R73, R74, R75, R76, R77, R78, R79, R8, R80, R81, R82, R83, R84, R85, R86, R87, R88, R89, R9, R90, R91, R92: footprint Resistor_THT:R_Axial_DIN0207_L6.3mm_D2.5mm_P7.62mm_Horizontal -> edited_footprints:R_Axial_DIN0207_L6.3mEDIT_m_D2.5mm_P7.62mm_Horizontal
- SW17: footprint Rotary_Encoder:RotaryEncoder_Alps_EC11E-Switch_Vertical_H20mm -> edited_footprints:EDIT_RotaryEncoder_Alps_EC11E-Switch_Vertical_H20mm

Commit message: Add files via upload
Parts:
- removed R1, R10, R11, R12, R13, R14, R15, R16, R18, R19, R2, R20, R21, R22, R23, R24, R25, R26, R27, R28, R29, R3, R30, R31, R32, R33, R34, R35, R36, R37, R38, R39, R4, R40, R41, R42, R43, R44, R45, R46, R47, R48, R49, R5, R50, R51, R52, R53, R54, R55, R56, R57, R58, R59, R6, R60, R61, R62, R63, R64, R65, R66, R67, R68, R69, R7, R70, R71, R72, R73, R74, R75, R76, R77, R78, R79, R8, R80, R81, R82, R83, R84, R85, R86, R87, R88, R89, R9, R90, R91, R92: RLED, edited_footprints:R_Axial_DIN0207_L6.3mEDIT_m_D2.5mm_P7.62mm_Horizontal, symbol Device:R
- D1, D10, D11, D12, D13, D14, D15, D16, D17, D18, D19, D2, D20, D21, D22, D23, D24, D25, D26, D27, D28, D29, D3, D30, D31, D32, D33, D34, D35, D36, D37, D38, D39, D4, D40, D41, D42, D43, D44, D45, D46, D47, D48, D49, D5, D50, D51, D52, D53, D54, D55, D56, D57, D58, D59, D6, D60, D61, D62, D63, D64, D65, D66, D67, D68, D69, D7, D70, D71, D72, D73, D74, D75, D76, D77, D78, D79, D8, D80, D81, D82, D83, D84, D85, D86, D87, D88, D89, D9, D90, D91, D92: footprint Diode_THT:D_DO-35_SOD27_P7.62mm_Horizontal -> Diode_THT:D_T-1_P5.08mm_Horizontal
Connections:
- net LED_0_OUT: now also SW1.3 (K), SW10.3 (K), SW11.3 (K), SW12.3 (K), SW13.3 (K), SW14.3 (K), SW15.3 (K), SW2.3 (K), SW3.3 (K), SW4.3 (K), SW5.3 (K), SW6.3 (K), SW7.3 (K), SW8.3 (K), SW9.3 (K); no longer U1.16 (GP12)
- net LED_1_OUT: now also SW16.3 (K), SW18.3 (K), SW19.3 (K), SW20.3 (K), SW21.3 (K), SW22.3 (K), SW23.3 (K), SW24.3 (K), SW25.3 (K), SW26.3 (K), SW27.3 (K), SW28.3 (K), SW29.3 (K), SW30.3 (K), SW31.3 (K), SW32.3 (K)
- net LED_2_OUT: now also SW33.3 (K), SW36.3 (K), SW37.3 (K), SW38.3 (K), SW39.3 (K), SW40.3 (K), SW41.3 (K), SW42.3 (K), SW43.3 (K), SW44.3 (K), SW45.3 (K), SW46.3 (K), SW47.3 (K), SW48.3 (K), SW49.3 (K)
- net LED_3_OUT: now also SW34.3 (K), SW35.3 (K), SW50.3 (K), SW51.3 (K), SW52.3 (K), SW53.3 (K), SW54.3 (K), SW55.3 (K), SW56.3 (K), SW57.3 (K), SW58.3 (K), SW59.3 (K), SW60.3 (K), SW61.3 (K), SW62.3 (K)
- net LED_4_OUT: now also SW63.3 (K), SW64.3 (K), SW67.3 (K), SW68.3 (K), SW69.3 (K), SW70.3 (K), SW71.3 (K), SW72.3 (K), SW73.3 (K), SW74.3 (K), SW75.3 (K), SW76.3 (K), SW77.3 (K), SW78.3 (K), SW79.3 (K)
- net LED_5_OUT: now also SW65.3 (K), SW66.3 (K), SW80.3 (K), SW81.3 (K), SW82.3 (K), SW83.3 (K), SW84.3 (K), SW85.3 (K), SW86.3 (K), SW87.3 (K), SW88.3 (K), SW89.3 (K), SW90.3 (K), SW91.3 (K), SW92.3 (K)
- net col12: now reaches SW13.2, SW30.2, SW46.2, SW88.2
- net col12: now also U1.16 (GP12)

Commit message: Add files via upload
Connections:
- net row0: now also U1.32 (GP28); no longer U1.26 (GP20)
- net row1: now also U1.31 (GP27); no longer U1.27 (GP21)
- net row2: now also U1.30 (GP26); no longer U1.29 (GP22)
- net row3: now also U1.29 (GP22); no longer U1.30 (GP26)
- net row4: now also U1.27 (GP21); no longer U1.31 (GP27)
- net row5: now also U1.26 (GP20); no longer U1.32 (GP28)
Changed lines of the file:
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@@
     (effects (font (size 1.27 1.27)) (justify right bottom))
   )
-  (label "row3" (at 210.82 311.15 0)
+  (label "row3" (at 210.82 313.69 0)
     (effects (font (size 1.27 1.27)) (justify left bottom))
   )
@@
     (effects (font (size 1.27 1.27)) (justify right bottom))
   )
-  (label "row0" (at 210.82 321.31 0)
+  (label "row0" (at 210.82 306.07 0)
     (effects (font (size 1.27 1.27)) (justify left bottom))
   )
@@
     (effects (font (size 1.27 1.27)) (justify right bottom))
   )
-  (label "row2" (at 210.82 313.69 0)
+  (label "row2" (at 210.82 311.15 0)
     (effects (font (size 1.27 1.27)) (justify left bottom))
   )
@@
     (effects (font (size 1.27 1.27)) (justify left bottom))
   )
-  (label "row4" (at 210.82 308.61 0)
+  (label "row4" (at 210.82 318.77 0)
     (effects (font (size 1.27 1.27)) (justify left bottom))
   )
@@
     (effects (font (size 1.27 1.27)) (justify right bottom))
   )
-  (label "row5" (at 210.82 306.07 0)
+  (label "row5" (at 210.82 321.31 0)
     (effects (font (size 1.27 1.27)) (justify left bottom))
   )
@@
     (effects (font (size 1.27 1.27)) (justify right bottom))
   )
-  (label "row1" (at 210.82 318.77 0)
-    (effects (font (size 1.27 1.27)) (justify left bottom))
-  )
+  (label "row1" (at 210.82 308.61 0)
+    (effects (font (size 1.27 1.27)) (justify left bottom))
+  )
