File: TKLC_v1/tklc_v1/tklc_v1.kicad_sch (KiCad schematic)
At the start: 200 parts, among them J1 UART breakout for extension b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, J2 RGB Strip breakout, J3 Encoder breakout, SW1 CherryMX_LED, SW10 CherryMX_LED, SW11 CherryMX_LED, SW12 CherryMX_LED, SW13 CherryMX_LED, SW14 CherryMX_LED, SW15 CherryMX_LED, SW16 CherryMX_LED, SW17 RotaryEncoder_Switch, SW18 CherryMX_LED, SW19 CherryMX_LED, SW2 CherryMX_LED, SW20 CherryMX_LED, SW21 CherryMX_LED, SW22 CherryMX_LED, SW23 CherryMX_LED, SW24 CherryMX_LED, SW25 CherryMX_LED, SW26 CherryMX_LED, SW27 CherryMX_LED, SW28 CherryMX_LED, SW29 CherryMX_LED, SW3 CherryMX_LED, SW30 CherryMX_LED, SW31 CherryMX_LED, SW32 CherryMX_LED, SW33 CherryMX_LED, SW34 CherryMX_LED, SW35 CherryMX_LED, SW36 CherryMX_LED, SW37 CherryMX_LED, SW38 CherryMX_LED, SW39 CherryMX_LED, SW4 CherryMX_LED, SW40 CherryMX_LED, SW41 CherryMX_LED, SW42 CherryMX_LED, SW43 CherryMX_LED, SW44 CherryMX_LED, SW45 CherryMX_LED, SW46 CherryMX_LED, SW47 CherryMX_LED, SW48 CherryMX_LED, SW49 CherryMX_LED, SW5 CherryMX_LED, SW50 CherryMX_LED, SW51 CherryMX_LED, SW52 CherryMX_LED, SW53 CherryMX_LED, SW54 CherryMX_LED, SW55 CherryMX_LED, SW56 CherryMX_LED, SW57 CherryMX_LED, SW58 CherryMX_LED, SW59 CherryMX_LED, SW6 CherryMX_LED, SW60 CherryMX_LED, SW61 CherryMX_LED, SW62 CherryMX_LED, SW63 CherryMX_LED, SW64 CherryMX_LED, SW65 CherryMX_LED, SW66 CherryMX_LED, SW67 CherryMX_LED, SW68 CherryMX_LED, SW69 CherryMX_LED, SW7 CherryMX_LED, SW70 CherryMX_LED, SW71 CherryMX_LED, SW72 CherryMX_LED, SW73 CherryMX_LED, SW74 CherryMX_LED, SW75 CherryMX_LED, SW76 CherryMX_LED, SW77 CherryMX_LED, SW78 CherryMX_LED, SW79 CherryMX_LED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

Commit message: Added SK6812 LEDs to schematic
Parts:
- removed J2: RGB Strip breakout, Connector:FanPinHeader_1x03_P2.54mm_Vertical, symbol Connector:Conn_01x03_Female
- removed U10, U11, U12, U13, U8, U9: MC34064P, Package_TO_SOT_THT:TO-92L_Inline, symbol Power_Supervisor:MC34064P
- D1, D10, D11, D12, D13, D14, D15, D16, D17, D18, D19, D2, D20, D21, D22, D23, D24, D25, D26, D27, D28, D29, D3, D30, D31, D32, D33, D34, D35, D36, D37, D38, D39, D4, D40, D41, D42, D43, D44, D45, D46, D47, D48, D49, D5, D50, D51, D52, D53, D54, D55, D56, D57, D58, D59, D6, D60, D61, D62, D63, D64, D65, D66, D67, D68, D69, D7, D70, D71, D72, D73, D74, D75, D76, D77, D78, D79, D8, D80, D81, D82, D83, D84, D85, D86, D87, D88, D89, D9, D90, D91, D92: footprint Diode_THT:D_T-1_P5.08mm_Horizontal -> Diode_THT:D_DO-35_SOD27_P7.62mm_Horizontal
- SW1, SW10, SW11, SW12, SW13, SW14, SW15, SW16, SW18, SW19, SW2, SW20, SW21, SW22, SW23, SW24, SW25, SW26, SW27, SW28, SW29, SW3, SW30, SW31, SW32, SW33, SW34, SW35, SW36, SW37, SW38, SW39, SW4, SW40, SW41, SW42, SW43, SW44, SW45, SW46, SW47, SW48, SW49, SW5, SW50, SW51, SW52, SW53, SW54, SW55, SW56, SW57, SW58, SW59, SW6, SW60, SW61, SW62, SW63, SW64, SW65, SW66, SW67, SW68, SW69, SW7, SW70, SW71, SW72, SW73, SW74, SW75, SW76, SW77, SW78, SW79, SW8, SW80, SW81, SW82, SW83, SW84, SW85, SW86, SW87, SW88, SW89, SW9, SW90, SW91, SW92: symbol Cherry MX:CherryMX_LED -> Cherry MX EDITS:CherryMX_SK6812
- renumbered J3 to J2
Connections:
- net GND: now also U2.3 (GND), U4.3 (GND), U6.3 (GND)
- net LED_0_IN: now also SW1.3 (VDD), SW10.3 (VDD), SW11.3 (VDD), SW12.3 (VDD), SW13.3 (VDD), SW14.3 (VDD), SW15.3 (VDD), SW16.3 (VDD), SW18.3 (VDD), SW19.3 (VDD), SW2.3 (VDD), SW20.3 (VDD), SW21.3 (VDD), SW22.3 (VDD), SW23.3 (VDD), SW24.3 (VDD), SW25.3 (VDD), SW26.3 (VDD), SW27.3 (VDD), SW28.3 (VDD), SW29.3 (VDD), SW3.3 (VDD), SW30.3 (VDD), SW31.3 (VDD), SW32.3 (VDD), SW33.3 (VDD), SW34.3 (VDD), SW35.3 (VDD), SW36.3 (VDD), SW37.3 (VDD), SW38.3 (VDD), SW39.3 (VDD), SW4.3 (VDD), SW40.3 (VDD), SW41.3 (VDD), SW42.3 (VDD), SW43.3 (VDD), SW44.3 (VDD), SW45.3 (VDD), SW46.3 (VDD), SW47.3 (VDD), SW48.3 (VDD), SW49.3 (VDD), SW5.3 (VDD), SW50.3 (VDD), SW51.3 (VDD), SW52.3 (VDD), SW53.3 (VDD), SW54.3 (VDD), SW55.3 (VDD), SW56.3 (VDD), SW57.3 (VDD), SW58.3 (VDD), SW59.3 (VDD), SW6.3 (VDD), SW60.3 (VDD), SW61.3 (VDD), SW62.3 (VDD), SW63.3 (VDD), SW64.3 (VDD), SW65.3 (VDD), SW66.3 (VDD), SW67.3 (VDD), SW68.3 (VDD), SW69.3 (VDD), SW7.3 (VDD), SW70.3 (VDD), SW71.3 (VDD), SW72.3 (VDD), SW73.3 (VDD), SW74.3 (VDD), SW75.3 (VDD), SW76.3 (VDD), SW77.3 (VDD), SW78.3 (VDD), SW79.3 (VDD), SW8.3 (VDD), SW80.3 (VDD), SW81.3 (VDD), SW82.3 (VDD), SW83.3 (VDD), SW84.3 (VDD), SW85.3 (VDD), SW86.3 (VDD), SW87.3 (VDD), SW88.3 (VDD), SW89.3 (VDD), SW9.3 (VDD), SW90.3 (VDD), SW91.3 (VDD), SW92.3 (VDD), U1.39 (VSYS); no longer SW1.4 (A), SW10.4 (A), SW11.4 (A), SW12.4 (A), SW13.4 (A), SW14.4 (A), SW15.4 (A), SW2.4 (A), SW3.4 (A), SW4.4 (A), SW5.4 (A), SW6.4 (A), SW7.4 (A), SW8.4 (A), SW9.4 (A), U2.3 (GND)
- net LED_0_OUT: now also SW1.6 (GND), SW10.6 (GND), SW11.6 (GND), SW12.6 (GND), SW13.6 (GND), SW14.6 (GND), SW15.6 (GND), SW2.6 (GND), SW3.6 (GND), SW4.6 (GND), SW5.6 (GND), SW6.6 (GND), SW7.6 (GND), SW8.6 (GND), SW9.6 (GND), U2.1 (~{RESET}); no longer SW1.3 (K), SW10.3 (K), SW11.3 (K), SW12.3 (K), SW13.3 (K), SW14.3 (K), SW15.3 (K), SW2.3 (K), SW3.3 (K), SW4.3 (K), SW5.3 (K), SW6.3 (K), SW7.3 (K), SW8.3 (K), SW9.3 (K), U3.1 (~{RESET})
- net LED_1_OUT: now also SW16.6 (GND), SW18.6 (GND), SW19.6 (GND), SW20.6 (GND), SW21.6 (GND), SW22.6 (GND), SW23.6 (GND), SW24.6 (GND), SW25.6 (GND), SW26.6 (GND), SW27.6 (GND), SW28.6 (GND), SW29.6 (GND), SW30.6 (GND), SW31.6 (GND), SW32.6 (GND), U3.1 (~{RESET}); no longer SW16.3 (K), SW18.3 (K), SW19.3 (K), SW20.3 (K), SW21.3 (K), SW22.3 (K), SW23.3 (K), SW24.3 (K), SW25.3 (K), SW26.3 (K), SW27.3 (K), SW28.3 (K), SW29.3 (K), SW30.3 (K), SW31.3 (K), SW32.3 (K), U5.1 (~{RESET})
- net LED_2_OUT: now also SW33.6 (GND), SW36.6 (GND), SW37.6 (GND), SW38.6 (GND), SW39.6 (GND), SW40.6 (GND), SW41.6 (GND), SW42.6 (GND), SW43.6 (GND), SW44.6 (GND), SW45.6 (GND), SW46.6 (GND), SW47.6 (GND), SW48.6 (GND), SW49.6 (GND), U4.1 (~{RESET}); no longer SW33.3 (K), SW36.3 (K), SW37.3 (K), SW38.3 (K), SW39.3 (K), SW40.3 (K), SW41.3 (K), SW42.3 (K), SW43.3 (K), SW44.3 (K), SW45.3 (K), SW46.3 (K), SW47.3 (K), SW48.3 (K), SW49.3 (K), U7.1 (~{RESET})
- net LED_3_OUT: now also SW34.6 (GND), SW35.6 (GND), SW50.6 (GND), SW51.6 (GND), SW52.6 (GND), SW53.6 (GND), SW54.6 (GND), SW55.6 (GND), SW56.6 (GND), SW57.6 (GND), SW58.6 (GND), SW59.6 (GND), SW60.6 (GND), SW61.6 (GND), SW62.6 (GND), U5.1 (~{RESET}); no longer SW34.3 (K), SW35.3 (K), SW50.3 (K), SW51.3 (K), SW52.3 (K), SW53.3 (K), SW54.3 (K), SW55.3 (K), SW56.3 (K), SW57.3 (K), SW58.3 (K), SW59.3 (K), SW60.3 (K), SW61.3 (K), SW62.3 (K)
- net LED_4_OUT: now also SW63.6 (GND), SW64.6 (GND), SW67.6 (GND), SW68.6 (GND), SW69.6 (GND), SW70.6 (GND), SW71.6 (GND), SW72.6 (GND), SW73.6 (GND), SW74.6 (GND), SW75.6 (GND), SW76.6 (GND), SW77.6 (GND), SW78.6 (GND), SW79.6 (GND), U6.1 (~{RESET}); no longer SW63.3 (K), SW64.3 (K), SW67.3 (K), SW68.3 (K), SW69.3 (K), SW70.3 (K), SW71.3 (K), SW72.3 (K), SW73.3 (K), SW74.3 (K), SW75.3 (K), SW76.3 (K), SW77.3 (K), SW78.3 (K), SW79.3 (K)
- net LED_5_OUT: now also SW65.6 (GND), SW66.6 (GND), SW80.6 (GND), SW81.6 (GND), SW82.6 (GND), SW83.6 (GND), SW84.6 (GND), SW85.6 (GND), SW86.6 (GND), SW87.6 (GND), SW88.6 (GND), SW89.6 (GND), SW90.6 (GND), SW91.6 (GND), SW92.6 (GND), U7.1 (~{RESET}); no longer SW65.3 (K), SW66.3 (K), SW80.3 (K), SW81.3 (K), SW82.3 (K), SW83.3 (K), SW84.3 (K), SW85.3 (K), SW86.3 (K), SW87.3 (K), SW88.3 (K), SW89.3 (K), SW90.3 (K), SW91.3 (K), SW92.3 (K)
- net LED_CONTROL: no longer U3.2 (IN), U5.2 (IN), U7.2 (IN)
- net RGB_DATA: now also SW1.4 (DIN)
- net row1: now also U3.2 (IN); no longer U4.2 (IN)
- net row2: now also U4.2 (IN); no longer U6.2 (IN)
- net row3: now also U5.2 (IN)
- net row4: now also U6.2 (IN)
- net row5: now also U7.2 (IN)
- removed net LED_1_IN: SW16.4 (A), SW18.4 (A), SW19.4 (A), SW20.4 (A), SW21.4 (A), SW22.4 (A), SW23.4 (A), SW24.4 (A), SW25.4 (A), SW26.4 (A), SW27.4 (A), SW28.4 (A), SW29.4 (A), SW30.4 (A), SW31.4 (A), SW32.4 (A), U4.3 (GND)
- removed net LED_2_IN: SW33.4 (A), SW36.4 (A), SW37.4 (A), SW38.4 (A), SW39.4 (A), SW40.4 (A), SW41.4 (A), SW42.4 (A), SW43.4 (A), SW44.4 (A), SW45.4 (A), SW46.4 (A), SW47.4 (A), SW48.4 (A), SW49.4 (A), U6.3 (GND)
- removed net LED_3_IN: SW34.4 (A), SW35.4 (A), SW50.4 (A), SW51.4 (A), SW52.4 (A), SW53.4 (A), SW54.4 (A), SW55.4 (A), SW56.4 (A), SW57.4 (A), SW58.4 (A), SW59.4 (A), SW60.4 (A), SW61.4 (A), SW62.4 (A)
- removed net LED_4_IN: SW63.4 (A), SW64.4 (A), SW67.4 (A), SW68.4 (A), SW69.4 (A), SW70.4 (A), SW71.4 (A), SW72.4 (A), SW73.4 (A), SW74.4 (A), SW75.4 (A), SW76.4 (A), SW77.4 (A), SW78.4 (A), SW79.4 (A)
- removed net LED_5_IN: SW65.4 (A), SW66.4 (A), SW80.4 (A), SW81.4 (A), SW82.4 (A), SW83.4 (A), SW84.4 (A), SW85.4 (A), SW86.4 (A), SW87.4 (A), SW88.4 (A), SW89.4 (A), SW90.4 (A), SW91.4 (A), SW92.4 (A)
- removed net VSYS: U1.39 (VSYS), U2.1 (~{RESET}), U4.1 (~{RESET}), U6.1 (~{RESET})
- new net: SW60.5 (DOUT), SW61.4 (DIN)
- new net: SW61.5 (DOUT), SW62.4 (DIN)
- new net: SW49.5 (DOUT), SW50.4 (DIN)
- new net: SW50.5 (DOUT), SW51.4 (DIN)
- new net: SW18.5 (DOUT), SW19.4 (DIN)
- new net: SW19.5 (DOUT), SW20.4 (DIN)
- new net: SW62.5 (DOUT), SW63.4 (DIN)
- new net: SW39.5 (DOUT), SW40.4 (DIN)
- new net: SW40.5 (DOUT), SW41.4 (DIN)
- new net: SW13.5 (DOUT), SW14.4 (DIN)
- new net: SW14.5 (DOUT), SW15.4 (DIN)
- new net: SW79.5 (DOUT), SW80.4 (DIN)
- new net: SW80.5 (DOUT), SW81.4 (DIN)
- new net: SW43.5 (DOUT), SW44.4 (DIN)
- new net: SW44.5 (DOUT), SW45.4 (DIN)
- new net: SW41.5 (DOUT), SW42.4 (DIN)
- new net: SW42.5 (DOUT), SW43.4 (DIN)
- new net: SW84.5 (DOUT), SW85.4 (DIN)
- new net: SW85.5 (DOUT), SW86.4 (DIN)
- new net: SW51.5 (DOUT), SW52.4 (DIN)
- new net: SW63.5 (DOUT), SW64.4 (DIN)
- new net: SW64.5 (DOUT), SW65.4 (DIN)
- new net: SW2.5 (DOUT), SW3.4 (DIN)
- new net: SW3.5 (DOUT), SW4.4 (DIN)
- new net: SW24.5 (DOUT), SW25.4 (DIN)
- new net: SW25.5 (DOUT), SW26.4 (DIN)
- new net: SW78.5 (DOUT), SW79.4 (DIN)
- new net: SW81.5 (DOUT), SW82.4 (DIN)
- new net: SW38.5 (DOUT), SW39.4 (DIN)
- new net: SW10.5 (DOUT), SW11.4 (DIN)
- new net: SW11.5 (DOUT), SW12.4 (DIN)
- new net: SW33.5 (DOUT), SW34.4 (DIN)
- new net: SW34.5 (DOUT), SW35.4 (DIN)
- new net: SW15.5 (DOUT), SW16.4 (DIN)
- new net: SW68.5 (DOUT), SW69.4 (DIN)
- new net: SW69.5 (DOUT), SW70.4 (DIN)
- new net: SW27.5 (DOUT), SW28.4 (DIN)
- new net: SW28.5 (DOUT), SW29.4 (DIN)
- new net: SW76.5 (DOUT), SW77.4 (DIN)
- new net: SW77.5 (DOUT), SW78.4 (DIN)
- new net: SW87.5 (DOUT), SW88.4 (DIN)
- new net: SW88.5 (DOUT), SW89.4 (DIN)
- new net: SW57.5 (DOUT), SW58.4 (DIN)
- new net: SW58.5 (DOUT), SW59.4 (DIN)
- new net: SW37.5 (DOUT), SW38.4 (DIN)
- new net: SW89.5 (DOUT), SW90.4 (DIN)
- new net: SW90.5 (DOUT), SW91.4 (DIN)
- new net: SW83.5 (DOUT), SW84.4 (DIN)
- new net: SW26.5 (DOUT), SW27.4 (DIN)
- new net: SW73.5 (DOUT), SW74.4 (DIN)
- new net: SW74.5 (DOUT), SW75.4 (DIN)
- new net: SW55.5 (DOUT), SW56.4 (DIN)
- new net: SW56.5 (DOUT), SW57.4 (DIN)
- new net: SW75.5 (DOUT), SW76.4 (DIN)
- new net: SW86.5 (DOUT), SW87.4 (DIN)
- new net: SW59.5 (DOUT), SW60.4 (DIN)
- new net: SW1.5 (DOUT), SW2.4 (DIN)
- new net: SW20.5 (DOUT), SW21.4 (DIN)
- new net: SW30.5 (DOUT), SW31.4 (DIN)
- new net: SW31.5 (DOUT), SW32.4 (DIN)
- new net: SW7.5 (DOUT), SW8.4 (DIN)
- new net: SW8.5 (DOUT), SW9.4 (DIN)
- new net: SW65.5 (DOUT), SW66.4 (DIN)
- new net: SW66.5 (DOUT), SW67.4 (DIN)
- new net: SW23.5 (DOUT), SW24.4 (DIN)
- new net: SW47.5 (DOUT), SW48.4 (DIN)
- new net: SW48.5 (DOUT), SW49.4 (DIN)
- new net: SW70.5 (DOUT), SW71.4 (DIN)
- new net: SW67.5 (DOUT), SW68.4 (DIN)
- new net: SW72.5 (DOUT), SW73.4 (DIN)
- new net: SW53.5 (DOUT), SW54.4 (DIN)
- new net: SW54.5 (DOUT), SW55.4 (DIN)
- new net: SW29.5 (DOUT), SW30.4 (DIN)
- new net: SW71.5 (DOUT), SW72.4 (DIN)
- new net: SW10.4 (DIN), SW9.5 (DOUT)
- new net: SW52.5 (DOUT), SW53.4 (DIN)
- new net: SW82.5 (DOUT), SW83.4 (DIN)
- new net: SW35.5 (DOUT), SW36.4 (DIN)
- new net: SW21.5 (DOUT), SW22.4 (DIN)
- new net: SW32.5 (DOUT), SW33.4 (DIN)
- new net: SW91.5 (DOUT), SW92.4 (DIN)
- new net: SW36.5 (DOUT), SW37.4 (DIN)
- new net: SW45.5 (DOUT), SW46.4 (DIN)
- new net: SW4.5 (DOUT), SW5.4 (DIN)
- new net: SW12.5 (DOUT), SW13.4 (DIN)
- new net: SW5.5 (DOUT), SW6.4 (DIN)
- new net: SW22.5 (DOUT), SW23.4 (DIN)
- new net: SW6.5 (DOUT), SW7.4 (DIN)
- new net: SW16.5 (DOUT), SW18.4 (DIN)
- new net: SW46.5 (DOUT), SW47.4 (DIN)
Other:
- moved on the sheet: D1, D10, D11, D12, D13, D14, D15, D16, D17, D18, D19, D2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
