File: TKLC_v1/tklc_v1_rgb_LP/tklc_v1_rgb_LP.kicad_sch (KiCad schematic)
At the start: 187 parts, among them J1 UART breakout for extension b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, J2 Encoder breakout, SW1 CherryMX_LED, SW10 CherryMX_LED, SW11 CherryMX_LED, SW12 CherryMX_LED, SW13 CherryMX_LED, SW14 CherryMX_LED, SW15 CherryMX_LED, SW16 CherryMX_LED, SW17 RotaryEncoder_Switch, SW18 CherryMX_LED, SW19 CherryMX_LED, SW2 CherryMX_LED, SW20 CherryMX_LED, SW21 CherryMX_LED, SW22 CherryMX_LED, SW23 CherryMX_LED, SW24 CherryMX_LED, SW25 CherryMX_LED, SW26 CherryMX_LED, SW27 CherryMX_LED, SW28 CherryMX_LED, SW29 CherryMX_LED, SW3 CherryMX_LED, SW30 CherryMX_LED, SW31 CherryMX_LED, SW32 CherryMX_LED, SW33 CherryMX_LED, SW34 CherryMX_LED, SW35 CherryMX_LED, SW36 CherryMX_LED, SW37 CherryMX_LED, SW38 CherryMX_LED, SW39 CherryMX_LED, SW4 CherryMX_LED, SW40 CherryMX_LED, SW41 CherryMX_LED, SW42 CherryMX_LED, SW43 CherryMX_LED, SW44 CherryMX_LED, SW45 CherryMX_LED, SW46 CherryMX_LED, SW47 CherryMX_LED, SW48 CherryMX_LED, SW49 CherryMX_LED, SW5 CherryMX_LED, SW50 CherryMX_LED, SW51 CherryMX_LED, SW52 CherryMX_LED, SW53 CherryMX_LED, SW54 CherryMX_LED, SW55 CherryMX_LED, SW56 CherryMX_LED, SW57 CherryMX_LED, SW58 CherryMX_LED, SW59 CherryMX_LED, SW6 CherryMX_LED, SW60 CherryMX_LED, SW61 CherryMX_LED, SW62 CherryMX_LED, SW63 CherryMX_LED, SW64 CherryMX_LED, SW65 CherryMX_LED, SW66 CherryMX_LED, SW67 CherryMX_LED, SW68 CherryMX_LED, SW69 CherryMX_LED, SW7 CherryMX_LED, SW70 CherryMX_LED, SW71 CherryMX_LED, SW72 CherryMX_LED, SW73 CherryMX_LED, SW74 CherryMX_LED, SW75 CherryMX_LED, SW76 CherryMX_LED, SW77 CherryMX_LED, SW78 CherryMX_LED, SW79 CherryMX_LED, SW8 CherryMX_LED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

Commit message: Finished wiring LEDs and Matrix to each other
Parts:
- D1, D10, D11, D12, D13, D14, D15, D16, D17, D18, D19, D2, D20, D21, D22, D23, D24, D25, D26, D27, D28, D29, D3, D30, D31, D32, D33, D34, D35, D36, D37, D38, D39, D4, D40, D41, D42, D43, D44, D45, D46, D47, D48, D49, D5, D50, D51, D52, D53, D54, D55, D56, D57, D58, D59, D6, D60, D61, D62, D63, D64, D65, D66, D67, D68, D69, D7, D70, D71, D72, D73, D74, D75, D76, D77, D78, D79, D8, D80, D81, D82, D83, D84, D85, D86, D87, D88, D89, D9, D90, D91, D92: footprint Diode_THT:D_T-1_P5.08mm_Horizontal -> edited_footprints:D_T-1_P5.08mm_Horizontal
